Commit message: Add config, launch, rviz, urdf, worlds and CMake updates for my_bot

File: src/my_bot/urdf/robot.urdf.xacro (robot description, xacro)
@@ -1,21 +1,29 @@
 <?xml version="1.0"?>
 <robot name="my_mesh_robot" xmlns:xacro="http://www.ros.org/wiki/xacro">
+  <xacro:property name="base_link_name" value="base_link"/>
+  <xacro:property name="lidar_frame_name" value="lidar_link"/>
   <link name="base_footprint"/>
   <joint name="base_joint" type="fixed">
     <parent link="base_footprint"/>
-    <child link="base_link"/>
+    <child link="${base_link_name}"/>
     <origin xyz="0 0 0.1075" rpy="0 0 0"/>
   </joint>
-  <link name="base_link">
-    <visual>
-      <geometry><mesh filename="package://my_bot/meshes/base_link.STL"/></geometry>
-      <material name="grey"><color rgba="0.5 0.5 0.5 1"/></material>
-    </visual>
-    <collision>
-      <geometry><mesh filename="package://my_bot/meshes/base_link.STL"/></geometry>
+  <link name="${base_link_name}">
+    <visual>
+      <geometry>
+        <mesh filename="package://my_bot/meshes/base_link.STL"/>
+      </geometry>
+      <material name="grey">
+        <color rgba="0.5 0.5 0.5 1"/>
+      </material>
+    </visual>
+    <collision>
+      <geometry>
+        <mesh filename="package://my_bot/meshes/base_link.STL"/>
+      </geometry>
     </collision>
     <inertial>
       <mass value="40.0"/>
-      <inertia ixx="0.58" ixy="0.0" ixz="0.0" iyy="1.03" iyz="0.0" izz="1.49"/>
+      <inertia ixx="1.0" ixy="0.0" ixz="0.0" iyy="1.0" iyz="0.0" izz="1.0"/>
     </inertial>
   </link>
@@ -23,17 +31,23 @@
     <visual>
       <origin xyz="0 0 0" rpy="1.5708 0 0"/>
-      <geometry><mesh filename="package://my_bot/meshes/l_wheel.STL"/></geometry>
-      <material name="black"><color rgba="0 0 0 1"/></material>
-    </visual>
-    <collision>
-      <geometry><cylinder radius="0.1075" length="0.05"/></geometry>
+      <geometry>
+        <mesh filename="package://my_bot/meshes/l_wheel.STL"/>
+      </geometry>
+      <material name="black">
+        <color rgba="0 0 0 1"/>
+      </material>
+    </visual>
+    <collision>
+      <geometry>
+        <cylinder radius="0.1075" length="0.05"/>
+      </geometry>
     </collision>
     <inertial>
       <mass value="2.4"/>
-      <inertia ixx="0.005" ixy="0" ixz="0" iyy="0.01" iyz="0" izz="0.005"/>
+      <inertia ixx="0.01" ixy="0" ixz="0" iyy="0.01" iyz="0" izz="0.01"/>
     </inertial>
   </link>
   <joint name="left_wheel_joint" type="continuous">
-    <parent link="base_link"/>
+    <parent link="${base_link_name}"/>
     <child link="left_wheel"/>
     <origin xyz="0 0.281 0" rpy="-1.5708 0 0"/>
@@ -41,20 +55,29 @@
     <dynamics damping="1.0" friction="0.2"/>
   </joint>
+  <gazebo reference="left_wheel">
+    <collision><surface><friction><ode><mu>1.2</mu><mu2>1.2</mu2></ode></friction><contact><ode><kp>50000</kp><kd>1.0</kd></ode></contact></surface></collision>
+  </gazebo>
   <link name="right_wheel">
     <visual>
       <origin xyz="0 0 0" rpy="1.5708 0 0"/>
-      <geometry><mesh filename="package://my_bot/meshes/r_wheel.STL"/></geometry>
-      <material name="black"/>
-    </visual>
-    <collision>
-      <geometry><cylinder radius="0.1075" length="0.05"/></geometry>
+      <geometry>
+        <mesh filename="package://my_bot/meshes/r_wheel.STL"/>
+      </geometry>
+      <material name="black">
+        <color rgba="0 0 0 1"/>
+      </material>
+    </visual>
+    <collision>
+      <geometry>
+        <cylinder radius="0.1075" length="0.05"/>
+      </geometry>
     </collision>
     <inertial>
       <mass value="2.4"/>
-      <inertia ixx="0.005" ixy="0" ixz="0" iyy="0.01" iyz="0" izz="0.005"/>
+      <inertia ixx="0.01" ixy="0" ixz="0" iyy="0.01" iyz="0" izz="0.01"/>
     </inertial>
   </link>
   <joint name="right_wheel_joint" type="continuous">
-    <parent link="base_link"/>
+    <parent link="${base_link_name}"/>
     <child link="right_wheel"/>
     <origin xyz="0 -0.281 0" rpy="-1.5708 0 0"/>
@@ -62,150 +85,76 @@
     <dynamics damping="1.0" friction="0.2"/>
   </joint>
-  <!-- Friction / contact for wheels (important: on the link collision, not the joint) -->
-  <gazebo reference="left_wheel">
-    <collision>
-      <surface>
-        <friction>
-          <ode>
-            <mu>1.2</mu>
-            <mu2>1.2</mu2>
-          </ode>
-        </friction>
-        <contact>
-          <ode>
-            <kp>50000</kp>
-            <kd>1.0</kd>
-          </ode>
-        </contact>
-      </surface>
-    </collision>
-  </gazebo>
   <gazebo reference="right_wheel">
-    <collision>
-      <surface>
-        <friction>
-          <ode>
-            <mu>1.2</mu>
-            <mu2>1.2</mu2>
-          </ode>
-        </friction>
-        <contact>
-          <ode>
-            <kp>50000</kp>
-            <kd>1.0</kd>
-          </ode>
-        </contact>
-      </surface>
-    </collision>
+    <collision><surface><friction><ode><mu>1.2</mu><mu2>1.2</mu2></ode></friction><contact><ode><kp>50000</kp><kd>1.0</kd></ode></contact></surface></collision>
   </gazebo>
   <link name="front_caster">
     <visual>
-      <geometry><mesh filename="package://my_bot/meshes/f_castor.STL"/></geometry>
+      <geometry>
+        <mesh filename="package://my_bot/meshes/f_castor.STL"/>
+      </geometry>
       <material name="silver"><color rgba="0.8 0.8 0.8 1"/></material>
     </visual>
-    <collision>
-      <geometry><sphere radius="0.05"/></geometry>
-    </collision>
-    <inertial>
-      <mass value="0.2"/>
-      <inertia ixx="0.0001" ixy="0" ixz="0" iyy="0.0001" iyz="0" izz="0.0001"/>
-    </inertial>
+    <collision><geometry><sphere radius="0.05"/></geometry></collision>
+    <inertial><mass value="0.2"/><inertia ixx="0.0005" ixy="0" ixz="0" iyy="0.0005" iyz="0" izz="0.0005"/></inertial>
   </link>
   <joint name="front_caster_joint" type="fixed">
-    <parent link="base_link"/>
-    <child link="front_caster"/>
+    <parent link="${base_link_name}"/><child link="front_caster"/>
     <origin xyz="0.3075 0.045 -0.0575" rpy="0 0 0"/>
   </joint>
+  <gazebo reference="front_caster">
+    <collision><surface><friction><ode><mu>1.0</mu><mu2>1.0</mu2></ode></friction><contact><ode><kp>20000</kp><kd>0.5</kd></ode></contact></surface></collision>
+  </gazebo>
   <link name="back_caster">
     <visual>
-      <geometry><mesh filename="package://my_bot/meshes/r_castor.STL"/></geometry>
-      <material name="silver"/>
-    </visual>
-    <collision>
-      <geometry><sphere radius="0.05"/></geometry>
-    </collision>
-    <inertial>
-      <mass value="0.2"/>
-      <inertia ixx="0.0001" ixy="0" ixz="0" iyy="0.0001" iyz="0" izz="0.0001"/>
-    </inertial>
+      <geometry>
+        <mesh filename="package://my_bot/meshes/r_castor.STL"/>
+      </geometry>
+      <material name="silver"><color rgba="0.8 0.8 0.8 1"/></material>
+    </visual>
+    <collision><geometry><sphere radius="0.05"/></geometry></collision>
+    <inertial><mass value="0.2"/><inertia ixx="0.0005" ixy="0" ixz="0" iyy="0.0005" iyz="0" izz="0.0005"/></inertial>
   </link>
   <joint name="back_caster_joint" type="fixed">
-    <parent link="base_link"/>
-    <child link="back_caster"/>
+    <parent link="${base_link_name}"/><child link="back_caster"/>
     <origin xyz="-0.3075 -0.045 -0.0575" rpy="0 0 0"/>
   </joint>
-  <!-- Friction for caster links (caster should have contact friction, joints are fixed) -->
-  <gazebo reference="front_caster">
-    <collision>
-      <surface>
-        <friction>
-          <ode>
-            <mu>1.0</mu>
-            <mu2>1.0</mu2>
-          </ode>
-        </friction>
-        <contact>
-          <ode>
-            <kp>20000</kp>
-            <kd>0.5</kd>
-          </ode>
-        </contact>
-      </surface>
-    </collision>
-  </gazebo>
   <gazebo reference="back_caster">
-    <collision>
-      <surface>
-        <friction>
-          <ode>
-            <mu>1.0</mu>
-            <mu2>1.0</mu2>
-          </ode>
-        </friction>
-        <contact>
-          <ode>
-            <kp>20000</kp>
-            <kd>0.5</kd>
-          </ode>
-        </contact>
-      </surface>
-    </collision>
+    <collision><surface><friction><ode><mu>1.0</mu><mu2>1.0</mu2></ode></friction><contact><ode><kp>20000</kp><kd>0.5</kd></ode></contact></surface></collision>
   </gazebo>
   <link name="imu_link"/>
   <joint name="imu_joint" type="fixed">
-    <parent link="base_link"/>
-    <child link="imu_link"/>
+    <parent link="${base_link_name}"/><child link="imu_link"/>
     <origin xyz="0.0 0 0.068" rpy="0 0 0"/>
   </joint>
   <gazebo reference="imu_link">
     <sensor name="imu_sensor" type="imu">
-      <always_on>1</always_on>
-      <update_rate>100</update_rate>
-      <visualize>true</visualize>
-      <topic>imu</topic>
+      <always_on>1</always_on><update_rate>100</update_rate><topic>imu</topic>
+      <imu>
+        <angular_velocity><noise type="gaussian"><mean>0.0</mean><stddev>0.001</stddev></noise></angular_velocity>
+        <linear_acceleration><noise type="gaussian"><mean>0.0</mean><stddev>0.01</stddev></noise></linear_acceleration>
+      </imu>
     </sensor>
   </gazebo>
-  <link name="lidar_link">
+  <link name="${lidar_frame_name}">
     <visual>
       <origin xyz="0 0 -0.03" rpy="0 0 0"/>
-      <geometry><mesh filename="package://my_bot/meshes/lidar.STL"/></geometry>
+      <geometry>
+        <mesh filename="package://my_bot/meshes/lidar.STL"/>
+      </geometry>
       <material name="blue"><color rgba="0 0 1 1"/></material>
     </visual>
     <collision>
-       <origin xyz="0 0 -0.03" rpy="0 0 0"/>
+      <origin xyz="0 0 -0.03" rpy="0 0 0"/>
       <geometry><cylinder radius="0.055" length="0.0315"/></geometry>
     </collision>
-    <inertial>
-      <mass value="0.1"/>
-      <inertia ixx="0.0001" ixy="0" ixz="0" iyy="0.0001" iyz="0" izz="0.0001"/>
-    </inertial>
+    <inertial><mass value="0.1"/><inertia ixx="0.0002" ixy="0" ixz="0" iyy="0.0002" iyz="0" izz="0.0002"/></inertial>
   </link>
   <joint name="lidar_joint" type="fixed">
-    <parent link="base_link"/>
-    <child link="lidar_link"/>
+    <parent link="${base_link_name}"/><child link="${lidar_frame_name}"/>
     <origin xyz="0 0 0.250" rpy="0 0 0"/>
   </joint>
-  <gazebo reference="lidar_link">
+  <gazebo reference="${lidar_frame_name}">
     <sensor name="lidar" type="gpu_lidar">
+      <gz_frame_id>${lidar_frame_name}</gz_frame_id>
       <pose>0 0 0 0 0 0</pose>
       <topic>scan</topic>
@@ -213,15 +162,7 @@
       <ray>
         <scan>
-          <horizontal>
-            <samples>360</samples>
-            <resolution>1</resolution>
-            <min_angle>0.0</min_angle>
-            <max_angle>6.28319</max_angle>
-          </horizontal>
+          <horizontal><samples>360</samples><resolution>1</resolution><min_angle>0.0</min_angle><max_angle>6.28319</max_angle></horizontal>
         </scan>
-        <range>
-          <min>0.12</min>
-          <max>4.0</max>
-        </range>
+        <range><min>0.12</min><max>4.0</max></range>
       </ray>
       <visualize>true</visualize>
@@ -230,36 +171,26 @@
   <link name="camera_link">
     <visual>
-      <geometry><box size="0.05 0.05 0.05"/></geometry>
+      <geometry>
+        <mesh filename="package://my_bot/meshes/camera.STL"/>
+      </geometry>
       <material name="red"><color rgba="1 0 0 1"/></material>
     </visual>
   </link>
   <joint name="camera_joint" type="fixed">
-    <parent link="base_link"/>
-    <child link="camera_link"/>
+    <parent link="${base_link_name}"/><child link="camera_link"/>
     <origin xyz="0.25 0 0.1" rpy="0 0 0"/>
   </joint>
-  <link name="camera_link_optical"></link>
+  <link name="camera_link_optical"/>
   <joint name="camera_optical_joint" type="fixed">
-    <parent link="camera_link"/>
-    <child link="camera_link_optical"/>
-    <origin xyz="0 0 0" rpy="-1.5708 0 -1.5708"/>
-  </joint>
-  <gazebo reference="camera_link">
+    <parent link="camera_link"/><child link="camera_link_optical"/>
+    <origin xyz="0 0 0" rpy="0 -1.5708 0"/>
+  </joint>
+  <gazebo reference="camera_link_optical">
     <sensor name="camera" type="camera">
-      <pose>0 0 0 0 0 0</pose>
-      <visualize>true</visualize>
-      <update_rate>30</update_rate>
-      <topic>camera/image_raw</topic>
+      <pose>0 0 0 0 0 0</pose><visualize>true</visualize><update_rate>30</update_rate><topic>camera/image_raw</topic>
       <camera>
         <horizontal_fov>1.089</horizontal_fov>
-        <image>
-          <format>R8G8B8</format>
-          <width>640</width>
-          <height>480</height>
-        </image>
-        <clip>
-          <near>0.05</near>
-          <far>8.0</far>
-        </clip>
+        <image><format>R8G8B8</format><width>640</width><height>480</height></image>
+        <clip><near>0.05</near><far>8.0</far></clip>
       </camera>
     </sensor>
@@ -281,11 +212,5 @@
       <topic>joint_states</topic>
     </plugin>
-    <!-- <plugin
-      filename="gz-sim-sensors-system"
-      name="gz::sim::systems::Sensors">
-      <render_engine>ogre2</render_engine>
-    </plugin> -->
-    <plugin filename="gz-sim-imu-system" name="gz::sim::systems::Imu">
-    </plugin>
+    <plugin filename="gz-sim-imu-system" name="gz::sim::systems::Imu"/>
   </gazebo>
 </robot>
